File: Hardware/MacroPad.kicad_pcb (KiCad board)
At the start: 2 copper layers, 76 x 93 mm, 37 parts, among them J1 USB_C_Receptacle_USB2.0_16P, SW1 SW_Push, SW10 SW_Push, SW11 SW_Push, SW2 SW_Push, SW3 SW_Push, SW4 SW_Push, SW5 SW_Push, SW6 SW_Push, SW7 SW_Push, SW8 SW_Push, SW9 SW_Push, U1 RP2040, U2 W25Q16JVSS, U3 AP2112K-3.3, U4 USBLC6-2SC6, Y1 12Mhz

Commit message: Commit 35: Updated Schematic and PCB
Parts:
- Y1: footprint Crystal:Crystal_SMD_3215-2Pin_3.2x1.5mm -> Crystal:Crystal_SMD_3225-4Pin_3.2x2.5mm
- moved C2 0.27 mm to (113.8, 119.8)
- moved C1 0.13 mm to (107.5, 119.8)
Connections:
- C4 pad 1: +5V -> +3.3V
- C5 pad 1: +5V -> +3.3V
Routing:
- net +5V: track 67.2 -> 57.9 mm
- net +3.3V: track 184.6 -> 189.8 mm
- net Net-(U1-XOUT): track 12.9 -> 9.84 mm
- net Net-(U1-XIN): track 11.4 -> 10.4 mm
