File: Hardware/MacroPad.kicad_sch (KiCad schematic)
At the start: 37 parts, among them J1 USB_C_Receptacle_USB2.0_16P, SW1 SW_Push, SW10 SW_Push, SW11 SW_Push, SW2 SW_Push, SW3 SW_Push, SW4 SW_Push, SW5 SW_Push, SW6 SW_Push, SW7 SW_Push, SW8 SW_Push, SW9 SW_Push, U1 RP2040, U2 W25Q16JVSS, U3 AP2112K-3.3, U4 USBLC6-2SC6, Y1 12Mhz

Commit message: Commit 35: Updated Schematic and PCB
Parts:
- C1, C2: MPN (none) -> GRM1555C1H150JA01D; Manufacturer (none) -> Murata; Type (none) -> SMD
- C10, C11, C12, C13, C3, C5, C7: MPN (none) -> CL05B104KO5NNNC; Manufacturer (none) -> Samsung; Type (none) -> SMD
- C4, C6: MPN (none) -> CL21A106KAYNNNE; Manufacturer (none) -> Samsung; Type (none) -> SMD
- C8, C9: MPN (none) -> CL05A105KA5NQNC; Manufacturer (none) -> Samsung; Type (none) -> SMD
- F1: MPN (none) -> 1206L050YR; Manufacturer (none) -> Littelfuse; Type (none) -> SMD
- J1: MPN (none) -> USB4085-GF-A; Manufacturer (none) -> GCT; Type (none) -> SMD
- R1, R6: MPN (none) -> RC0402FR-0710KL; Manufacturer (none) -> Yageo; Type (none) -> SMD
- R2, R3: MPN (none) -> RC0402FR-075K1L; Manufacturer (none) -> Yageo; Type (none) -> SMD
- R4, R5: MPN (none) -> RC0402FR-0727RL; Manufacturer (none) -> Yageo; Type (none) -> SMD
- SW1, SW2, SW3, SW4, SW5, SW6, SW7, SW8, SW9: now not fitted
- SW10, SW11: MPN (none) -> PTS810 SJK 250 SMTR LFS; Manufacturer (none) -> C&K; Type (none) -> SMD
- U1: MPN (none) -> SC0914(13); Manufacturer (none) -> Raspberry Pi; Type (none) -> SMD
- U2: MPN (none) -> W25Q16JVSSIQ; Manufacturer (none) -> Winbond; Type (none) -> SMD
- U3: MPN (none) -> AP2112K-3.3TRG1; Manufacturer (none) -> Diodes Incorporated; Type (none) -> SMD
- U4: MPN (none) -> USBLC6-2SC6; Manufacturer (none) -> STMicroelectronics; Type (none) -> SMD
- Y1: footprint Crystal:Crystal_SMD_3215-2Pin_3.2x1.5mm -> Crystal:Crystal_SMD_3225-4Pin_3.2x2.5mm; MPN (none) -> ABM8-272-T3; Manufacturer (none) -> Abracon; Type (none) -> SMD
Connections:
- net +3.3V: now also C4.1, C5.1, U3.5 (VOUT)
- net +5V: no longer C4.1, C5.1, U3.5 (VOUT)
